File: hardware/AMP_RCv2.kicad_sch (KiCad schematic)
At the start: 47 parts, among them CN3 Conn_01x15, CN4 Conn_01x15, J1 USB_C_Receptacle_USB2.0_16P, SW1 SW_UP, SW2 SW_LEFT, SW3 SW_DOWN, SW4 SW_RIGHT, SW5 ON/OFF, U1 TPS61023, U2 MCP73831-2-OT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

Commit message: Finish routing
Parts:
- removed CN3, CN4: Conn_01x15, Connector_PinHeader_2.54mm:PinHeader_1x15_P2.54mm_Vertical, symbol Connector_Generic:Conn_01x15
- added U7: NUCLEO32-F303K8, AMP_Custom:NUCLEO32, symbol AMP_Custom:NUCLEO32-F303K8
Connections:
- net +3V3: now also U7.17 (+3V3)
- net +5V: now also U7.27 (+5V)
- net BAT_CHRG_STAT: now also U7.9 (PB1)
- net BUTTON_DOWN: now also U7.11 (PF1)
- net BUTTON_LEFT: now also U7.8 (PB6)
- net BUTTON_RIGHT: now also U7.21 (PA3)
- net BUTTON_UP: now also U7.7 (PB7)
- net GND: now also U7.29 (GND), U7.4 (GND)
- net JOYSTICK_LEFT_H: now also U7.19 (PA0)
- net JOYSTICK_LEFT_SW: now also U7.6 (PB0)
- net JOYSTICK_LEFT_V: now also U7.20 (PA1)
- net JOYSTICK_RIGHT_H: now also U7.23 (PA5)
- net JOYSTICK_RIGHT_SW: now also U7.12 (PA8)
- net JOYSTICK_RIGHT_V: now also U7.22 (PA4)
- net LORA_DIO0: now also U7.5 (PA12)
- net LORA_NSS: now also U7.2 (PA10)
- net LORA_RST: now also U7.1 (PA9)
- net OLED_DC: now also U7.14 (PB5)
- net OLED_NSS: now also U7.13 (PA11)
- net OLED_RST: now also U7.15 (PB4)
- net PA6 renamed SPI1_MISO
- net SPI1_MISO: now also U7.24 (PA6)
- net PA7 renamed SPI1_MOSI
- net SPI1_MOSI: now also U7.25 (PA7)
- net PB3 renamed SPI1_SCK
- net SPI1_SCK: now also U7.16 (PB3)
- new net: U7.28 (NRST), U7.3 (NRST)
- no-connect marks 15 -> 16
